File: kicad_schematic_files/shift_registers.sch (KiCad schematic (older format))
At the start: 28 parts, among them U10 74HC595, U11 74HC595, U12 74HC595, U13 74HC595, U14 74HC595, U15 74HC595, U16 74HC595, U17 74HC595, U4 74HC595, U5 74HC595, U6 74HC595, U7 74HC595, U8 74HC595, U9 74HC595

Commit message: v2 board
Parts:
- U10, U11, U12, U13, U14, U15, U16, U17, U4, U5, U6, U7, U8, U9: footprint Package_SO:SOIC-16W_7.5x10.3mm_P1.27mm -> Package_SO:SOIC-16_3.9x9.9mm_P1.27mm
Changed lines of the file:
@@
 $Descr USLetter 11000 8500
 encoding utf-8
-Sheet 2 6
+Sheet 6 6
 Title "Stepper Clock"
 Date "2021-09-17"
@@
 F 0 "U7" V 1900 5850 50  0000 L CNN
 F 1 "74HC595" V 2000 5750 50  0000 L CNN
-F 2 "Package_SO:SOIC-16W_7.5x10.3mm_P1.27mm" H 1900 5950 50  0001 C CNN
+F 2 "Package_SO:SOIC-16_3.9x9.9mm_P1.27mm" H 1900 5950 50  0001 C CNN
 F 3 "http://www.ti.com/lit/ds/symlink/sn74hc595.pdf" H 1900 5950 50  0001 C CNN
 	1    1900 5950
@@
 F 0 "U6" V 4250 5850 50  0000 L CNN
 F 1 "74HC595" V 4350 5750 50  0000 L CNN
-F 2 "Package_SO:SOIC-16W_7.5x10.3mm_P1.27mm" H 4250 5950 50  0001 C CNN
+F 2 "Package_SO:SOIC-16_3.9x9.9mm_P1.27mm" H 4250 5950 50  0001 C CNN
 F 3 "http://www.ti.com/lit/ds/symlink/sn74hc595.pdf" H 4250 5950 50  0001 C CNN
 	1    4250 5950
@@
 F 0 "U11" V 1900 4300 50  0000 L CNN
 F 1 "74HC595" V 2000 4200 50  0000 L CNN
-F 2 "Package_SO:SOIC-16W_7.5x10.3mm_P1.27mm" H 1900 4400 50  0001 C CNN
+F 2 "Package_SO:SOIC-16_3.9x9.9mm_P1.27mm" H 1900 4400 50  0001 C CNN
 F 3 "http://www.ti.com/lit/ds/symlink/sn74hc595.pdf" H 1900 4400 50  0001 C CNN
 	1    1900 4400
@@
 F 0 "U10" V 4250 4300 50  0000 L CNN
 F 1 "74HC595" V 4350 4200 50  0000 L CNN
-F 2 "Package_SO:SOIC-16W_7.5x10.3mm_P1.27mm" H 4250 4400 50  0001 C CNN
+F 2 "Package_SO:SOIC-16_3.9x9.9mm_P1.27mm" H 4250 4400 50  0001 C CNN
 F 3 "http://www.ti.com/lit/ds/symlink/sn74hc595.pdf" H 4250 4400 50  0001 C CNN
 	1    4250 4400
@@
 F 0 "U9" V 6550 4300 50  0000 L CNN
 F 1 "74HC595" V 6650 4200 50  0000 L CNN
-F 2 "Package_SO:SOIC-16W_7.5x10.3mm_P1.27mm" H 6550 4400 50  0001 C CNN
+F 2 "Package_SO:SOIC-16_3.9x9.9mm_P1.27mm" H 6550 4400 50  0001 C CNN
 F 3 "http://www.ti.com/lit/ds/symlink/sn74hc595.pdf" H 6550 4400 50  0001 C CNN
 	1    6550 4400
@@
 F 0 "U5" V 6550 5850 50  0000 L CNN
 F 1 "74HC595" V 6650 5750 50  0000 L CNN
-F 2 "Package_SO:SOIC-16W_7.5x10.3mm_P1.27mm" H 6550 5950 50  0001 C CNN
+F 2 "Package_SO:SOIC-16_3.9x9.9mm_P1.27mm" H 6550 5950 50  0001 C CNN
 F 3 "http://www.ti.com/lit/ds/symlink/sn74hc595.pdf" H 6550 5950 50  0001 C CNN
 	1    6550 5950
@@
 F 0 "U15" V 1900 2900 50  0000 L CNN
 F 1 "74HC595" V 2000 2800 50  0000 L CNN
-F 2 "Package_SO:SOIC-16W_7.5x10.3mm_P1.27mm" H 1900 3000 50  0001 C CNN
+F 2 "Package_SO:SOIC-16_3.9x9.9mm_P1.27mm" H 1900 3000 50  0001 C CNN
 F 3 "http://www.ti.com/lit/ds/symlink/sn74hc595.pdf" H 1900 3000 50  0001 C CNN
 	1    1900 3000
@@
 F 0 "U14" V 4250 2900 50  0000 L CNN
 F 1 "74HC595" V 4350 2800 50  0000 L CNN
-F 2 "Package_SO:SOIC-16W_7.5x10.3mm_P1.27mm" H 4250 3000 50  0001 C CNN
+F 2 "Package_SO:SOIC-16_3.9x9.9mm_P1.27mm" H 4250 3000 50  0001 C CNN
 F 3 "http://www.ti.com/lit/ds/symlink/sn74hc595.pdf" H 4250 3000 50  0001 C CNN
 	1    4250 3000
@@
 F 0 "U13" V 6550 2900 50  0000 L CNN
 F 1 "74HC595" V 6650 2800 50  0000 L CNN
-F 2 "Package_SO:SOIC-16W_7.5x10.3mm_P1.27mm" H 6550 3000 50  0001 C CNN
+F 2 "Package_SO:SOIC-16_3.9x9.9mm_P1.27mm" H 6550 3000 50  0001 C CNN
 F 3 "http://www.ti.com/lit/ds/symlink/sn74hc595.pdf" H 6550 3000 50  0001 C CNN
 	1    6550 3000
@@
 F 0 "U4" V 9100 5850 50  0000 L CNN
 F 1 "74HC595" V 9200 5750 50  0000 L CNN
-F 2 "Package_SO:SOIC-16W_7.5x10.3mm_P1.27mm" H 9100 5950 50  0001 C CNN
+F 2 "Package_SO:SOIC-16_3.9x9.9mm_P1.27mm" H 9100 5950 50  0001 C CNN
 F 3 "http://www.ti.com/lit/ds/symlink/sn74hc595.pdf" H 9100 5950 50  0001 C CNN
 	1    9100 5950
@@
 F 0 "U8" V 9100 4300 50  0000 L CNN
 F 1 "74HC595" V 9200 4200 50  0000 L CNN
-F 2 "Package_SO:SOIC-16W_7.5x10.3mm_P1.27mm" H 9100 4400 50  0001 C CNN
+F 2 "Package_SO:SOIC-16_3.9x9.9mm_P1.27mm" H 9100 4400 50  0001 C CNN
 F 3 "http://www.ti.com/lit/ds/symlink/sn74hc595.pdf" H 9100 4400 50  0001 C CNN
 	1    9100 4400
@@
 F 0 "U17" V 6550 1450 50  0000 L CNN
 F 1 "74HC595" V 6650 1350 50  0000 L CNN
-F 2 "Package_SO:SOIC-16W_7.5x10.3mm_P1.27mm" H 6550 1550 50  0001 C CNN
+F 2 "Package_SO:SOIC-16_3.9x9.9mm_P1.27mm" H 6550 1550 50  0001 C CNN
 F 3 "http://www.ti.com/lit/ds/symlink/sn74hc595.pdf" H 6550 1550 50  0001 C CNN
 	1    6550 1550
@@
 F 0 "U16" V 9100 1450 50  0000 L CNN
 F 1 "74HC595" V 9200 1350 50  0000 L CNN
-F 2 "Package_SO:SOIC-16W_7.5x10.3mm_P1.27mm" H 9100 1550 50  0001 C CNN
+F 2 "Package_SO:SOIC-16_3.9x9.9mm_P1.27mm" H 9100 1550 50  0001 C CNN
 F 3 "http://www.ti.com/lit/ds/symlink/sn74hc595.pdf" H 9100 1550 50  0001 C CNN
 	1    9100 1550
@@
 F 0 "U12" V 9100 2900 50  0000 L CNN
 F 1 "74HC595" V 9200 2800 50  0000 L CNN
-F 2 "Package_SO:SOIC-16W_7.5x10.3mm_P1.27mm" H 9100 3000 50  0001 C CNN
+F 2 "Package_SO:SOIC-16_3.9x9.9mm_P1.27mm" H 9100 3000 50  0001 C CNN
 F 3 "http://www.ti.com/lit/ds/symlink/sn74hc595.pdf" H 9100 3000 50  0001 C CNN
 	1    9100 3000
